File: PCB/lpkbv1/lpkbv1.kicad_sch (KiCad schematic)
At the start: 194 parts, among them J2 OLED_128x64, SW1 SW_Push_45deg, SW10 SW_Push_45deg, SW11 SW_Push_45deg, SW12 SW_Push_45deg, SW13 SW_Push_45deg, SW14 SW_Push_45deg, SW15 SW_Push_45deg, SW16 SW_Push_45deg, SW17 SW_Push_45deg, SW18 SW_Push_45deg, SW19 SW_Push_45deg, SW2 SW_Push_45deg, SW20 SW_Push_45deg, SW21 SW_Push_45deg, SW22 SW_Push_45deg, SW23 SW_Push_45deg, SW24 SW_Push_45deg, SW25 SW_Push_45deg, SW26 SW_Push_45deg, SW27 SW_Push_45deg, SW28 SW_Push_45deg, SW29 SW_Push_45deg, SW3 SW_Push_45deg, SW30 SW_Push_45deg, SW31 SW_Push_45deg, SW32 SW_Push_45deg, SW33 SW_Push_45deg, SW34 SW_Push_45deg, SW35 SW_Push_45deg, SW36 SW_Push_45deg, SW37 SW_Push_45deg, SW38 SW_Push_45deg, SW39 SW_Push_45deg, SW4 SW_Push_45deg, SW40 SW_Push_45deg, SW41 SW_Push_45deg, SW42 SW_Push_45deg, SW43 SW_Push_45deg, SW44 SW_Push_45deg, SW45 SW_Push_45deg, SW46 SW_Push_45deg, SW47 SW_Push_45deg, SW48 SW_Push_45deg, SW49 SW_Push_45deg, SW5 SW_Push_45deg, SW50 SW_Push_45deg, SW51 SW_Push_45deg, SW52 SW_Push_45deg, SW53 SW_Push_45deg, SW54 SW_Push_45deg, SW55 SW_Push_45deg, SW56 SW_Push_45deg, SW57 SW_Push_45deg, SW58 SW_Push_45deg, SW59 SW_Push_45deg, SW6 SW_Push_45deg, SW60 SW_Push_45deg, SW61 SW_Push_45deg, SW62 SW_Push_45deg, SW63 SW_Push_45deg, SW64 SW_Push_45deg, SW65 SW_Push_45deg, SW66 SW_Push_45deg, SW67 SW_Push_45deg, SW68 SW_Push_45deg, SW69 SW_Push_45deg, SW7 SW_Push_45deg, SW70 SW_Push_45deg, SW71 SW_Push_45deg, SW72 SW_Push_45deg, SW73 SW_Push_45deg, SW74 SW_Push_45deg, SW75 SW_Push_45deg, SW76 SW_Push_45deg, SW77 SW_Push_45deg, SW78 SW_Push_45deg, SW79 SW_Push_45deg, SW8 SW_Push_45deg, SW80 SW_Push_45deg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

Commit message: Ship ready!
Parts:
- SW1, SW10, SW11, SW12, SW13, SW14, SW15, SW16, SW17, SW18, SW19, SW2, SW20, SW21, SW22, SW23, SW24, SW25, SW26, SW27, SW28, SW29, SW3, SW30, SW31, SW32, SW33, SW34, SW35, SW36, SW37, SW38, SW39, SW4, SW40, SW41, SW42, SW43, SW44, SW45, SW46, SW47, SW48, SW49, SW5, SW50, SW51, SW52, SW53, SW54, SW55, SW56, SW57, SW58, SW59, SW6, SW60, SW61, SW62, SW63, SW64, SW65, SW66, SW67, SW68, SW69, SW7, SW70, SW71, SW72, SW73, SW74, SW75, SW76, SW77, SW78, SW79, SW8, SW80, SW81, SW82, SW83, SW84, SW85, SW86, SW87, SW88, SW89, SW9: footprint lib:SW_Gateron_LowProfile_THT -> lib:SW_MX_LowProfile_THT

Commit message: Firmware fix + gerber fix
Parts:
- removed C1, C2: 4.7U, Capacitor_SMD:C_0402_1005Metric, symbol Device:C
- removed C3: 10u, Capacitor_SMD:C_0402_1005Metric, symbol Device:C
- removed D83, D84, D85: LED, LED_THT:LED_D1.8mm_W3.3mm_H2.4mm, symbol Device:LED
- removed R10: 1k, Resistor_SMD:R_0402_1005Metric, symbol Device:R
- removed R3, R9: 10k, Resistor_SMD:R_0402_1005Metric, symbol Device:R
- removed R4, R5, R6: 470, Resistor_SMD:R_0402_1005Metric, symbol Device:R
- removed R7: 330K, Resistor_SMD:R_0402_1005Metric, symbol Device:R
- removed R8: 110K, Resistor_SMD:R_0402_1005Metric, symbol Device:R
- removed U1: MCP73871, Package_DFN_QFN:QFN-20-1EP_4x4mm_P0.5mm_EP2.5x2.5mm, symbol Battery_Management:MCP73871
- added D83, D84: D_Schottky, Diode_THT:D_DO-41_SOD81_P7.62mm_Horizontal, symbol Device:D_Schottky
- added J1: Output, Connector_PinHeader_2.54mm:PinHeader_1x02_P2.54mm_Vertical, symbol Connector_Generic:Conn_01x02
- added J3: Charge, Connector_PinHeader_2.54mm:PinHeader_1x02_P2.54mm_Vertical, symbol Connector_Generic:Conn_01x02
- added R1: 200K, Resistor_THT:R_Axial_DIN0204_L3.6mm_D1.6mm_P7.62mm_Horizontal, symbol Device:R
- added R2: 100K, Resistor_THT:R_Axial_DIN0204_L3.6mm_D1.6mm_P7.62mm_Horizontal, symbol Device:R
- added SW90, SW91: SW_SPDT, Connector_PinHeader_1.00mm:PinHeader_1x03_P1.00mm_Vertical, symbol Switch:SW_SPDT
- BT1: footprint Battery:BatteryHolder_Keystone_1042_1x18650 -> Connector_PinHeader_2.54mm:PinHeader_1x02_P2.54mm_Vertical
Connections:
- net GND: now also J1.1 (Pin_1), J3.1 (Pin_1), R1.1, SW91.3 (C)
- net VSYS: now also SW90.2 (B), SW91.1 (A)
- net at BT1.1 (+): now also R2.2
- net BAT_SENSE: now reaches A1.34 (GPIO28_ADC2)
- net BAT_SENSE: now also R1.2, R2.1
- net 3v3_EN: now reaches A1.37 (3V3_EN)
- net 3v3_EN: now also SW91.2 (B)
- new net: D84.2 (A), J1.2 (Pin_2)
- new net: D83.1 (K), J3.2 (Pin_2)
- new net: D84.1 (K), SW90.1 (A)
- new net: D83.2 (A), SW90.3 (C)
- no-connect marks 4 -> 2
Other:
- note added: "Charge Select"
